Commit message: Transform Fix

File: wheelchair_description/urdf/urdf.urdf (robot description, URDF)
Before this commit: robot wheelchair, 5 links, 4 joints
Links:
- added link base_footprint
Joints:
- added joint connector: type fixed, parent base_footprint, child base_link, origin xyz=0 0 0 rpy=1.57 0 3.14
- joint camera: origin xyz=-0.39931 0.33074 -0.35378 rpy=3.1416 1.5708 0 -> xyz=-0.39931 0.33074 -0.35378 rpy=1.5708 0 -3.1416
- joint lidar_joint: origin xyz=-0.64132 -0.14701 -0.37178 rpy=1.5714 1.5708 0 -> xyz=-0.64132 -0.14701 -0.37178 rpy=1.5708 0 -3.1416

Commit message: Transforms fix 2

File: wheelchair_description/urdf/urdf.urdf (robot description, URDF)
Before this commit: robot wheelchair, 6 links, 5 joints
Links:
- removed link base_footprint
- added link chassis, mass 9.6593; collision mesh filename=package://wheelchair_description/meshes/base_link.STL; visual mesh filename=package://wheelchair_description/meshes/base_link.STL
- link base_link: mass 9.6593 -> None; geometry 
Joints:
- joint camera: parent base_link -> chassis
- joint connector: child base_link -> chassis; parent base_footprint -> base_link
- joint lidar_joint: origin xyz=-0.64132 -0.14701 -0.37178 rpy=1.5708 0 -3.1416 -> xyz=-0.64132 -0.14701 -0.37178 rpy=1.5714 1.5708 0; parent base_link -> chassis
- joint wheel1: parent base_link -> chassis
- joint wheel2: parent base_link -> chassis

Commit message: Camera Fix

File: wheelchair_description/urdf/urdf.urdf (robot description, URDF)
Before this commit: robot wheelchair, 6 links, 5 joints
Links:
- added link camera_link
Joints:
- added joint camera_link_gazebo: type fixed, parent chassis, child camera_link, origin xyz=-0.39931 0.33074 -0.35378 rpy=1.5708 0 -3.1416, axis 0 0 0
- joint camera: origin xyz=-0.39931 0.33074 -0.35378 rpy=1.5708 0 -3.1416 -> xyz=0 0 0 rpy=-1.5708 0 -1.5708; parent chassis -> camera_link
- joint connector: origin xyz=0 0 0 rpy=1.57 0 3.14 -> xyz=0 0 0.4 rpy=1.57 0 3.14

Commit message: Port fix

File: wheelchair_description/urdf/urdf.urdf (robot description, URDF)
Before this commit: robot wheelchair, 7 links, 6 joints
Links:
- added link lidar_link, mass 0.13016; collision mesh filename=package://wheelchair_description/meshes/lidar.STL; visual mesh filename=package://wheelchair_description/meshes/lidar.STL
- link lidar: mass 0.13016 -> None; geometry 
Joints:
- added joint lidar_link_geometry: type fixed, parent lidar_link, child lidar, origin xyz=0 0 0 rpy=-3.1416 0 -1.5708, axis 0 0 0
- joint lidar_joint: child lidar -> lidar_link

Commit message: Base footprint update

File: wheelchair_description/urdf/urdf.urdf (robot description, URDF)
Before this commit: robot wheelchair, 8 links, 7 joints
Links:
- added link base_footprint
Joints:
- added joint base_link_footprint: type fixed, parent base_link, child base_footprint, origin xyz=0 0 -0.4 rpy=0 0 0
- joint connector: origin xyz=0 0 0.4 rpy=1.57 0 3.14 -> xyz=0 0 0 rpy=1.57 0 3.14
- joint lidar_link_geometry: origin xyz=0 0 0 rpy=-3.1416 0 -1.5708 -> xyz=0 0 0 rpy=0 0 -3.1416

Commit message: Odom Fix

File: wheelchair_description/urdf/urdf.urdf (robot description, URDF)
Before this commit: robot wheelchair, 9 links, 8 joints
Links:
- removed link lidar
- added link laser
Joints:
- joint lidar_link_geometry: child lidar -> laser; origin xyz=0 0 0 rpy=0 0 -3.1416 -> xyz=0 0 0 rpy=0 0 3.1416
